File: Electronics/lightboxschematicv2.brd (EAGLE design)
At the start: 35.5 x 44.1 mm, 13 parts, among them IC1 ATMEGA328-PU, SW1 FSM8JRT, U1 LT1085CT-5PBF

Commit message: Add files via upload
Connections:
- new net N$5: IC1.15, R4.1
Routing:
- net N$5: track 0.00 -> 35.6 mm
Changed lines of the file:
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@@
 <wire x1="52.1208" y1="67.056" x2="52.07" y2="67.31" width="0.3048" layer="1"/>
+</signal>
+<signal name="N$5">
+<contactref element="IC1" pad="15"/>
+<contactref element="R4" pad="1"/>
+<wire x1="34.925" y1="37.465" x2="34.925" y2="44.45" width="0.3048" layer="1"/>
+<wire x1="39.6875" y1="32.7025" x2="34.925" y2="37.465" width="0.3048" layer="1"/>
+<wire x1="59.69" y1="32.7025" x2="39.6875" y2="32.7025" width="0.3048" layer="1"/>
+<wire x1="59.69" y1="34.29" x2="59.69" y2="32.7025" width="0.3048" layer="1"/>
+<wire x1="34.925" y1="44.45" x2="34.61" y2="44.45" width="0.3048" layer="1"/>
 </signal>
 </signals>
