File: Electronics/lightboxschematicv2.sch (EAGLE design)
At the start: 13 parts, among them IC1 ATMEGA328-PU, SW1 FSM8JRT, U1 LT1085CT-5PBF

Commit message: Add files via upload
Connections:
- new net N$5: IC1.(OC1A)PB1, R4.1
Other:
- moved on the sheet: R4
Changed lines of the file:
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@@
 <attribute name="VALUE" x="168.9148" y="81.785440625" size="1.780240625" layer="96" rot="R90"/>
 </instance>
-<instance part="R4" gate="G$1" x="154.94" y="93.98">
-<attribute name="NAME" x="151.12403125" y="95.989740625" size="1.78078125" layer="95"/>
-<attribute name="VALUE" x="151.122209375" y="90.41673125" size="1.781640625" layer="96"/>
+<instance part="R4" gate="G$1" x="157.48" y="93.98">
+<attribute name="NAME" x="153.66403125" y="95.989740625" size="1.78078125" layer="95"/>
+<attribute name="VALUE" x="153.662209375" y="90.41673125" size="1.781640625" layer="96"/>
 </instance>
 <instance part="R5" gate="G$1" x="99.06" y="104.14" rot="R90">
@@
 <net name="N$2" class="0">
 <segment>
-<wire x1="160.02" y1="93.98" x2="162.56" y2="93.98" width="0.1524" layer="91"/>
+<wire x1="162.56" y1="93.98" x2="165.1" y2="93.98" width="0.1524" layer="91"/>
 <pinref part="D1" gate="G$1" pin="A"/>
 <pinref part="R4" gate="G$1" pin="2"/>
-<wire x1="162.56" y1="93.98" x2="165.1" y2="93.98" width="0.1524" layer="91"/>
-<junction x="162.56" y="93.98"/>
+<junction x="165.1" y="93.98"/>
 </segment>
 </net>
@@
 </segment>
 </net>
+<net name="N$5" class="0">
+<segment>
+<pinref part="IC1" gate="IC" pin="(OC1A)PB1"/>
+<pinref part="R4" gate="G$1" pin="1"/>
+</segment>
+</net>
